Commit message: One publisching of joint_states and status

File: wsg50_description/urdf/wsg50_210_macro.urdf.xacro (robot description, xacro)
@@ -19,4 +19,10 @@
          </geometry>
       </visual>
+      <visual>
+        <origin xyz="0 0 0" rpy="0 0 0" />
+        <geometry>
+            <mesh filename="package://wsg50_description/meshes/black_plate.dae" />
+         </geometry>
+      </visual>
       <collision>
         <origin xyz="0 0 0" rpy="0 0 0" />
@@ -25,10 +31,4 @@
         </geometry>
       </collision>
-      <visual>
-        <origin xyz="0 0 0" rpy="0 0 0" />
-        <geometry>
-            <mesh filename="package://wsg50_description/meshes/black_plate.dae" />
-         </geometry>
-      </visual>
     </link>
     <joint name="${name}_finger_left_joint" type="prismatic" >

Commit message: Updated launch files, description and size definition as parameter

File: wsg50_description/urdf/wsg50_210_macro.urdf.xacro (robot description, xacro)
@@ -1,5 +1,5 @@
 <?xml version="1.0"?>
 <robot  xmlns:xacro="http://www.ros.org/wiki/xacro">
-  <xacro:macro name="wsg50_210" params="name parent *origin">
+  <xacro:macro name="wsg50" params="name parent *origin">
     <joint name="${name}_palm_joint" type="fixed">
         <insert_block name="origin"/>
@@ -16,5 +16,5 @@
         <origin xyz="0 0 0" rpy="0 0 0" />
         <geometry>
-            <mesh filename="package://wsg50_description/meshes/palm.dae" />
+            <mesh filename="package://wsg50_description/meshes/palm_210.dae" />
          </geometry>
       </visual>
@@ -28,5 +28,5 @@
         <origin xyz="0 0 0" rpy="0 0 0" />
         <geometry>
-            <mesh filename="package://wsg50_description/meshes/palm.stl" scale="0.001 0.001 0.001" />
+            <mesh filename="package://wsg50_description/meshes/palm_210.stl" scale="0.001 0.001 0.001" />
         </geometry>
       </collision>
