Commit message: Update names

File: wsg50_description/urdf/wsg50_210.urdf.xacro (robot description, xacro)
@@ -2,5 +2,5 @@
 <!--Generates a urdf from the macro in kr16_2_macro.xacro -->
 <robot name="wsg50_210" xmlns:xacro="http://www.ros.org/wiki/xacro">
-  <xacro:include filename="$(find schunk_description)/urdf/common.xacro" />
+  <xacro:property name="M_PI" value="3.1415926535897931" />
   <link name="world"/>
   <xacro:include filename="$(find wsg50_description)/urdf/wsg50_210_macro.urdf.xacro" />

File: wsg50_description/urdf/wsg50_210_macro.urdf.xacro (robot description, xacro)
@@ -1,5 +1,5 @@
 <?xml version="1.0"?>
 <robot  xmlns:xacro="http://www.ros.org/wiki/xacro">
-  <xacro:macro name="wsg50" params="name parent *origin">
+  <xacro:macro name="wsg50_210" params="name parent *origin">
     <joint name="${name}_palm_joint" type="fixed">
         <insert_block name="origin"/>

Commit message: Updated xacro

File: wsg50_description/urdf/wsg50_210.urdf.xacro (robot description, xacro)
@@ -2,5 +2,4 @@
 <!--Generates a urdf from the macro in kr16_2_macro.xacro -->
 <robot name="wsg50_210" xmlns:xacro="http://www.ros.org/wiki/xacro">
-  <xacro:property name="M_PI" value="3.1415926535897931" />
   <link name="world"/>
   <xacro:include filename="$(find wsg50_description)/urdf/wsg50_210_macro.urdf.xacro" />

File: wsg50_description/urdf/wsg50_210_macro.urdf.xacro (robot description, xacro)
@@ -3,5 +3,5 @@
   <xacro:macro name="wsg50_210" params="name parent *origin">
     <joint name="${name}_palm_joint" type="fixed">
-        <insert_block name="origin"/>
+        <xacro:insert_block name="origin"/>
         <parent link="${parent}"/>
         <child link="${name}_palm_link"/>
@@ -59,5 +59,5 @@
     </link>
     <joint name="${name}_finger_right_joint" type="prismatic" >
-      <origin xyz="0 0 0.0719" rpy="0 0 ${M_PI}"/>
+      <origin xyz="0 0 0.0719" rpy="0 0 ${pi}"/>
       <parent link="${name}_palm_link" />
       <child link="${name}_finger_right_link" />
